Commit message: changed scale to 0.1

File: RJJE_Arm/rjje_arm_ws/src/rjje_arm/urdf/definitions.xacro (robot description, xacro)
@@ -17,9 +17,9 @@
       <inertial>
         <mass value="${mass}" />
-        <origin rpy="${origin_rpy}" xyz="${origin_xyz}" />
+        <origin rpy="${origin_rpy}" xyz="${float(origin_xyz.split(' ')[0])*0.1} ${float(origin_xyz.split(' ')[1])*0.1} ${float(origin_xyz.split(' ')[2])*0.1}" />
         <inertia ixx="${ixx}" ixy="${ixy}" ixz="${ixz}" iyy="${iyy}" iyz="${iyz}" izz="${izz}" />
       </inertial>
       <collision>
-        <origin rpy="${origin_rpy}" xyz="${origin_xyz}" />
+        <origin rpy="${origin_rpy}" xyz="${float(origin_xyz.split(' ')[0])*0.1} ${float(origin_xyz.split(' ')[1])*0.1} ${float(origin_xyz.split(' ')[2])*0.1}" />
         <geometry>
           <mesh filename="${meshfile}" scale="${meshscale}"/>
@@ -27,5 +27,5 @@
       </collision>
       <visual>
-        <origin rpy="${origin_rpy}" xyz="${origin_xyz}" />
+        <origin rpy="${origin_rpy}" xyz="${float(origin_xyz.split(' ')[0])*0.1} ${float(origin_xyz.split(' ')[1])*0.1} ${float(origin_xyz.split(' ')[2])*0.1}" />
         <geometry>
           <mesh filename="${meshfile}" scale="${meshscale}"/>
@@ -39,5 +39,5 @@
       <axis xyz="${axis_xyz}"/>
       <limit effort="${limit_e}" lower="${limit_l}" upper="${limit_u}" velocity="${limit_v}" />
-      <origin rpy="${origin_rpy}" xyz="${origin_xyz}"/>
+      <origin rpy="${origin_rpy}" xyz="${float(origin_xyz.split(' ')[0])*0.1} ${float(origin_xyz.split(' ')[1])*0.1} ${float(origin_xyz.split(' ')[2])*0.1}"/>
       <parent link="${parent}" />
       <child link="${child}"/>
@@ -48,5 +48,5 @@
       <axis xyz="${axis_xyz}"/>
       <limit effort="${limit_e}" lower="${limit_l}" upper="${limit_u}" velocity="${limit_v}" />
-      <origin rpy="${origin_rpy}" xyz="${origin_xyz}"/>
+      <origin rpy="${origin_rpy}" xyz="${float(origin_xyz.split(' ')[0])*0.1} ${float(origin_xyz.split(' ')[1])*0.1} ${float(origin_xyz.split(' ')[2])*0.1}"/>
       <parent link="${parent}" />
       <child link="${child}"/>
@@ -57,5 +57,5 @@
     <link name="${name}">
       <visual>
-        <origin xyz="${origin_xyz}" rpy="${origin_rpy}"/>
+        <origin xyz="${float(origin_xyz.split(' ')[0])*0.1} ${float(origin_xyz.split(' ')[1])*0.1} ${float(origin_xyz.split(' ')[2])*0.1}" rpy="${origin_rpy}"/>
         <geometry>
             <cylinder length="${length}" radius="${radius}"/>
@@ -64,5 +64,5 @@
       </visual>
       <collision>
-          <origin xyz="${origin_xyz}" rpy="${origin_rpy}"/>
+          <origin xyz="${float(origin_xyz.split(' ')[0])*0.1} ${float(origin_xyz.split(' ')[1])*0.1} ${float(origin_xyz.split(' ')[2])*0.1}" rpy="${origin_rpy}"/>
           <geometry>
               <cylinder length="${length}" radius="${radius}"/>

File: RJJE_Arm/rjje_arm_ws/src/rjje_arm/urdf/rjje_arm.xacro (robot description, xacro)
@@ -12,5 +12,5 @@
     origin_rpy="0.0 0.0 0.0"
     meshfile="package://rjje_arm/meshes/base.stl"
-    meshscale="0.01 0.01 0.01"
+    meshscale="0.1 0.1 0.1"
     mass="1.57633"
     ixx="0.13235" ixy="0" ixz="0"
@@ -32,5 +32,5 @@
     origin_rpy="0.0 0.0 0.0"
     meshfile="package://rjje_arm/meshes/motor_and_frame.stl"
-    meshscale="0.01 0.01 0.01"
+    meshscale="0.1 0.1 0.1"
     mass="1.57633"
     ixx="0.13235" ixy="0" ixz="0"
@@ -52,5 +52,5 @@
     origin_rpy="0.0 0.0 3.14"
     meshfile="package://rjje_arm/meshes/thin_bracket.stl"
-    meshscale="0.01 0.01 0.01"
+    meshscale="0.1 0.1 0.1"
     mass="1.57633"
     ixx="0.13235" ixy="0" ixz="0"
@@ -72,5 +72,5 @@
     origin_rpy="0.0 0.0 0.0"
     meshfile="package://rjje_arm/meshes/motor_and_frame.stl"
-    meshscale="0.01 0.01 0.01"
+    meshscale="0.1 0.1 0.1"
     mass="1.57633"
     ixx="0.13235" ixy="0" ixz="0"
@@ -92,5 +92,5 @@
     origin_rpy="0.0 0.0 0.0"
     meshfile="package://rjje_arm/meshes/thin_bracket.stl"
-    meshscale="0.01 0.01 0.01"
+    meshscale="0.1 0.1 0.1"
     mass="1.57633"
     ixx="0.13235" ixy="0" ixz="0"
@@ -112,5 +112,5 @@
     origin_rpy="0.0 0.0 0.0"
     meshfile="package://rjje_arm/meshes/thin_bracket.stl"
-    meshscale="0.01 0.01 0.01"
+    meshscale="0.1 0.1 0.1"
     mass="1.57633"
     ixx="0.13235" ixy="0" ixz="0"
@@ -132,5 +132,5 @@
     origin_rpy="0.0 0.0 0.0"
     meshfile="package://rjje_arm/meshes/motor_and_frame.stl"
-    meshscale="0.01 0.01 0.01"
+    meshscale="0.1 0.1 0.1"
     mass="1.57633"
     ixx="0.13235" ixy="0" ixz="0"
@@ -169,5 +169,5 @@
     origin_rpy="0.0 0.0 0.0"
     meshfile="package://rjje_arm/meshes/thin_bracket.stl"
-    meshscale="0.01 0.01 0.01"
+    meshscale="0.1 0.1 0.1"
     mass="1.57633"
     ixx="0.13235" ixy="0" ixz="0"
@@ -189,5 +189,5 @@
     origin_rpy="0.0 0.0 0.0"
     meshfile="package://rjje_arm/meshes/motor_and_frame.stl"
-    meshscale="0.01 0.01 0.01"
+    meshscale="0.1 0.1 0.1"
     mass="1.57633"
     ixx="0.13235" ixy="0" ixz="0"
@@ -209,5 +209,5 @@
     origin_rpy="0.0 0.0 0.0"
     meshfile="package://rjje_arm/meshes/motor_and_frame.stl"
-    meshscale="0.01 0.01 0.01"
+    meshscale="0.1 0.1 0.1"
     mass="1.57633"
     ixx="0.13235" ixy="0" ixz="0"
@@ -249,5 +249,5 @@
     origin_rpy="0.0 0.0 0.0"
     meshfile="package://rjje_arm/meshes/gripper_finger.stl"
-    meshscale="0.01 0.01 0.01"
+    meshscale="0.1 0.1 0.1"
     mass="1.57633"
     ixx="0.13235" ixy="0" ixz="0"
@@ -269,5 +269,5 @@
     origin_rpy="0.0 0.0 0.0"
     meshfile="package://rjje_arm/meshes/gripper_finger.stl"
-    meshscale="0.01 0.01 0.01"
+    meshscale="0.1 0.1 0.1"
     mass="1.57633"
     ixx="0.13235" ixy="0" ixz="0"

File: RJJE_Arm/rjje_arm_ws/src/rjje_arm/urdf/rjje_arm.xacro.urdf (robot description, URDF)
Before this commit: robot rjje_arm, 15 links, 14 joints
Links:
- link base_link: geometry collision mesh filename=package://rjje_arm/meshes/base.stl scale=0.1 0.1 0.1; visual mesh filename=package://rjje_arm/meshes/base.stl scale=0.1 0.1 0.1
- link bracket_1: geometry collision mesh filename=package://rjje_arm/meshes/thin_bracket.stl scale=0.1 0.1 0.1; visual mesh filename=package://rjje_arm/meshes/thin_bracket.stl scale=0.1 0.1 0.1
- link bracket_2_1: geometry collision mesh filename=package://rjje_arm/meshes/thin_bracket.stl scale=0.1 0.1 0.1; visual mesh filename=package://rjje_arm/meshes/thin_bracket.stl scale=0.1 0.1 0.1
- link bracket_2_2: geometry collision mesh filename=package://rjje_arm/meshes/thin_bracket.stl scale=0.1 0.1 0.1; visual mesh filename=package://rjje_arm/meshes/thin_bracket.stl scale=0.1 0.1 0.1
- link bracket_3_2: geometry collision mesh filename=package://rjje_arm/meshes/thin_bracket.stl scale=0.1 0.1 0.1; visual mesh filename=package://rjje_arm/meshes/thin_bracket.stl scale=0.1 0.1 0.1
- link left_gripper: geometry collision mesh filename=package://rjje_arm/meshes/gripper_finger.stl scale=0.1 0.1 0.1; visual mesh filename=package://rjje_arm/meshes/gripper_finger.stl scale=0.1 0.1 0.1
- link link1: geometry collision mesh filename=package://rjje_arm/meshes/motor_and_frame.stl scale=0.1 0.1 0.1; visual mesh filename=package://rjje_arm/meshes/motor_and_frame.stl scale=0.1 0.1 0.1
- link link_2: geometry collision mesh filename=package://rjje_arm/meshes/motor_and_frame.stl scale=0.1 0.1 0.1; visual mesh filename=package://rjje_arm/meshes/motor_and_frame.stl scale=0.1 0.1 0.1
- link link_3: geometry collision mesh filename=package://rjje_arm/meshes/motor_and_frame.stl scale=0.1 0.1 0.1; visual mesh filename=package://rjje_arm/meshes/motor_and_frame.stl scale=0.1 0.1 0.1
- link link_4: geometry collision mesh filename=package://rjje_arm/meshes/motor_and_frame.stl scale=0.1 0.1 0.1; visual mesh filename=package://rjje_arm/meshes/motor_and_frame.stl scale=0.1 0.1 0.1
- link link_5: geometry collision mesh filename=package://rjje_arm/meshes/motor_and_frame.stl scale=0.1 0.1 0.1; visual mesh filename=package://rjje_arm/meshes/motor_and_frame.stl scale=0.1 0.1 0.1
- link right_gripper: geometry collision mesh filename=package://rjje_arm/meshes/gripper_finger.stl scale=0.1 0.1 0.1; visual mesh filename=package://rjje_arm/meshes/gripper_finger.stl scale=0.1 0.1 0.1
Joints:
- joint base_link_link1: origin xyz=3.45 4.2 4.0 rpy=0 0 0 -> xyz=0.34500000000000003 0.42000000000000004 0.4 rpy=0 0 0
- joint bracket_1_link_2: origin xyz=2.2 0.0 1.4 rpy=1.57 0.0 -1.57 -> xyz=0.22000000000000003 0.0 0.13999999999999999 rpy=1.57 0.0 -1.57
- joint bracket_2_1_bracket_2_2: origin xyz=0.0 10.5 0.0 rpy=0.0 0.0 3.14 -> xyz=0.0 1.05 0.0 rpy=0.0 0.0 3.14
- joint bracket_2_2_link_3: origin xyz=0.0 0.0 -5.3 rpy=0.0 0.0 3.14 -> xyz=0.0 0.0 -0.53 rpy=0.0 0.0 3.14
- joint bracket_3_1_bracket_3_2: origin xyz=-2.65 0.0 6.75 rpy=-1.57 0.0 1.57 -> xyz=-0.265 0.0 0.675 rpy=-1.57 0.0 1.57
- joint bracket_3_2_link_4: origin xyz=0.0 0.0 -5.3 rpy=0.0 0.0 -1.57 -> xyz=0.0 0.0 -0.53 rpy=0.0 0.0 -1.57
- joint link1_bracket_1: origin xyz=0 0 5.3 rpy=0 0 0 -> xyz=0.0 0.0 0.53 rpy=0 0 0
- joint link_2_bracket_2_1: origin xyz=0.0 0.0 5.3 rpy=0.0 0.0 0.0 -> xyz=0.0 0.0 0.53 rpy=0.0 0.0 0.0
- joint link_3_bracket_3_1: origin xyz=4.0 0.0 2.0 rpy=0.0 1.57 0.0 -> xyz=0.4 0.0 0.2 rpy=0.0 1.57 0.0
- joint link_4_link_5: origin xyz=0.0 2.4 2.2 rpy=0.0 1.57 0.0 -> xyz=0.0 0.24 0.22000000000000003 rpy=0.0 1.57 0.0
- joint link_5_link_6: origin xyz=0.0 0.0 5.2 rpy=0.0 0.0 0.0 -> xyz=0.0 0.0 0.52 rpy=0.0 0.0 0.0
- joint link_6_left_gripper: origin xyz=-1.6 0.0 1.6 rpy=1.57 0.0 0.0 -> xyz=-0.16000000000000003 0.0 0.16000000000000003 rpy=1.57 0.0 0.0
- joint link_6_right_gripper: origin xyz=1.6 0.0 1.6 rpy=1.57 0.0 0.0 -> xyz=0.16000000000000003 0.0 0.16000000000000003 rpy=1.57 0.0 0.0
- joint world_base_link: origin xyz=0 0 0.0 rpy=0 0 0 -> xyz=0.0 0.0 0.0 rpy=0 0 0

Commit message: fixed urdf!

File: RJJE_Arm/rjje_arm_ws/src/rjje_arm/urdf/definitions.xacro (robot description, xacro)
@@ -13,4 +13,5 @@
     <color rgba="0.2 0.2 0.1 1.0"/>
   </material>
+  <xacro:property name="scale_factor" value="0.01" />
   <!-- Note on xyz: this is just a string. and {} means to eval -->
   <xacro:macro name="m_link_mesh" params="name origin_xyz origin_rpy meshfile meshscale mass ixx ixy ixz iyy iyz izz color">
@@ -18,9 +19,9 @@
       <inertial>
         <mass value="${mass}" />
-        <origin rpy="${origin_rpy}" xyz="${float(origin_xyz.split(' ')[0])*0.1} ${float(origin_xyz.split(' ')[1])*0.1} ${float(origin_xyz.split(' ')[2])*0.1}" />
+        <origin rpy="${origin_rpy}" xyz="${float(origin_xyz.split(' ')[0])*scale_factor} ${float(origin_xyz.split(' ')[1])*scale_factor} ${float(origin_xyz.split(' ')[2])*scale_factor}" />
         <inertia ixx="${ixx}" ixy="${ixy}" ixz="${ixz}" iyy="${iyy}" iyz="${iyz}" izz="${izz}" />
       </inertial>
       <collision>
-        <origin rpy="${origin_rpy}" xyz="${float(origin_xyz.split(' ')[0])*0.1} ${float(origin_xyz.split(' ')[1])*0.1} ${float(origin_xyz.split(' ')[2])*0.1}" />
+        <origin rpy="${origin_rpy}" xyz="${float(origin_xyz.split(' ')[0])*scale_factor} ${float(origin_xyz.split(' ')[1])*scale_factor} ${float(origin_xyz.split(' ')[2])*scale_factor}" />
         <geometry>
           <mesh filename="${meshfile}" scale="${meshscale}"/>
@@ -28,5 +29,5 @@
       </collision>
       <visual>
-        <origin rpy="${origin_rpy}" xyz="${float(origin_xyz.split(' ')[0])*0.1} ${float(origin_xyz.split(' ')[1])*0.1} ${float(origin_xyz.split(' ')[2])*0.1}" />
+        <origin rpy="${origin_rpy}" xyz="${float(origin_xyz.split(' ')[0])*scale_factor} ${float(origin_xyz.split(' ')[1])*scale_factor} ${float(origin_xyz.split(' ')[2])*scale_factor}" />
         <geometry>
           <mesh filename="${meshfile}" scale="${meshscale}"/>
@@ -40,5 +41,5 @@
       <axis xyz="${axis_xyz}"/>
       <limit effort="${limit_e}" lower="${limit_l}" upper="${limit_u}" velocity="${limit_v}" />
-      <origin rpy="${origin_rpy}" xyz="${float(origin_xyz.split(' ')[0])*0.1} ${float(origin_xyz.split(' ')[1])*0.1} ${float(origin_xyz.split(' ')[2])*0.1}"/>
+      <origin rpy="${origin_rpy}" xyz="${float(origin_xyz.split(' ')[0])*scale_factor} ${float(origin_xyz.split(' ')[1])*scale_factor} ${float(origin_xyz.split(' ')[2])*scale_factor}"/>
       <parent link="${parent}" />
       <child link="${child}"/>
@@ -49,5 +50,5 @@
       <axis xyz="${axis_xyz}"/>
       <limit effort="${limit_e}" lower="${limit_l}" upper="${limit_u}" velocity="${limit_v}" />
-      <origin rpy="${origin_rpy}" xyz="${float(origin_xyz.split(' ')[0])*0.1} ${float(origin_xyz.split(' ')[1])*0.1} ${float(origin_xyz.split(' ')[2])*0.1}"/>
+      <origin rpy="${origin_rpy}" xyz="${float(origin_xyz.split(' ')[0])*scale_factor} ${float(origin_xyz.split(' ')[1])*scale_factor} ${float(origin_xyz.split(' ')[2])*scale_factor}"/>
       <parent link="${parent}" />
       <child link="${child}"/>
@@ -58,14 +59,14 @@
     <link name="${name}">
       <visual>
-        <origin xyz="${float(origin_xyz.split(' ')[0])*0.1} ${float(origin_xyz.split(' ')[1])*0.1} ${float(origin_xyz.split(' ')[2])*0.1}" rpy="${origin_rpy}"/>
+        <origin xyz="${float(origin_xyz.split(' ')[0])*scale_factor} ${float(origin_xyz.split(' ')[1])*scale_factor} ${float(origin_xyz.split(' ')[2])*scale_factor}" rpy="${origin_rpy}"/>
         <geometry>
-            <cylinder length="${length}" radius="${radius}"/>
+            <cylinder length="${length *scale_factor }" radius="${radius *scale_factor }"/>
          </geometry>
          <material name="${color}"/>
       </visual>
       <collision>
-          <origin xyz="${float(origin_xyz.split(' ')[0])*0.1} ${float(origin_xyz.split(' ')[1])*0.1} ${float(origin_xyz.split(' ')[2])*0.1}" rpy="${origin_rpy}"/>
+          <origin xyz="${float(origin_xyz.split(' ')[0])*scale_factor} ${float(origin_xyz.split(' ')[1])*scale_factor} ${float(origin_xyz.split(' ')[2])*scale_factor}" rpy="${origin_rpy}"/>
           <geometry>
-              <cylinder length="${length}" radius="${radius}"/>
+              <cylinder length="${length *scale_factor }" radius="${radius *scale_factor }"/>
           </geometry>
       </collision>

File: RJJE_Arm/rjje_arm_ws/src/rjje_arm/urdf/rjje_arm.xacro (robot description, xacro)
@@ -7,4 +7,5 @@
   <link name="world">
   </link>
+  <!-- scale_factor is defined in definitions.xacro -->
   <xacro:m_link_mesh
     name="base_link"
@@ -12,5 +13,5 @@
     origin_rpy="0.0 0.0 0.0"
     meshfile="package://rjje_arm/meshes/base.stl"
-    meshscale="0.1 0.1 0.1"
+    meshscale="${scale_factor} ${scale_factor} ${scale_factor}"
     mass="1.57633"
     ixx="0.13235" ixy="0" ixz="0"
@@ -32,5 +33,5 @@
     origin_rpy="0.0 0.0 0.0"
     meshfile="package://rjje_arm/meshes/motor_and_frame.stl"
-    meshscale="0.1 0.1 0.1"
+    meshscale="${scale_factor} ${scale_factor} ${scale_factor}"
     mass="1.57633"
     ixx="0.13235" ixy="0" ixz="0"
@@ -52,5 +53,5 @@
     origin_rpy="0.0 0.0 3.14"
     meshfile="package://rjje_arm/meshes/thin_bracket.stl"
-    meshscale="0.1 0.1 0.1"
+    meshscale="${scale_factor} ${scale_factor} ${scale_factor}"
     mass="1.57633"
     ixx="0.13235" ixy="0" ixz="0"
@@ -72,5 +73,5 @@
     origin_rpy="0.0 0.0 0.0"
     meshfile="package://rjje_arm/meshes/motor_and_frame.stl"
-    meshscale="0.1 0.1 0.1"
+    meshscale="${scale_factor} ${scale_factor} ${scale_factor}"
     mass="1.57633"
     ixx="0.13235" ixy="0" ixz="0"
@@ -92,5 +93,5 @@
     origin_rpy="0.0 0.0 0.0"
     meshfile="package://rjje_arm/meshes/thin_bracket.stl"
-    meshscale="0.1 0.1 0.1"
+    meshscale="${scale_factor} ${scale_factor} ${scale_factor}"
     mass="1.57633"
     ixx="0.13235" ixy="0" ixz="0"
@@ -112,5 +113,5 @@
     origin_rpy="0.0 0.0 0.0"
     meshfile="package://rjje_arm/meshes/thin_bracket.stl"
-    meshscale="0.1 0.1 0.1"
+    meshscale="${scale_factor} ${scale_factor} ${scale_factor}"
     mass="1.57633"
     ixx="0.13235" ixy="0" ixz="0"
@@ -132,5 +133,5 @@
     origin_rpy="0.0 0.0 0.0"
     meshfile="package://rjje_arm/meshes/motor_and_frame.stl"
-    meshscale="0.1 0.1 0.1"
+    meshscale="${scale_factor} ${scale_factor} ${scale_factor}"
     mass="1.57633"
     ixx="0.13235" ixy="0" ixz="0"
@@ -169,5 +170,5 @@
     origin_rpy="0.0 0.0 0.0"
     meshfile="package://rjje_arm/meshes/thin_bracket.stl"
-    meshscale="0.1 0.1 0.1"
+    meshscale="${scale_factor} ${scale_factor} ${scale_factor}"
     mass="1.57633"
     ixx="0.13235" ixy="0" ixz="0"
@@ -189,5 +190,5 @@
     origin_rpy="0.0 0.0 0.0"
     meshfile="package://rjje_arm/meshes/motor_and_frame.stl"
-    meshscale="0.1 0.1 0.1"
+    meshscale="${scale_factor} ${scale_factor} ${scale_factor}"
     mass="1.57633"
     ixx="0.13235" ixy="0" ixz="0"
@@ -209,5 +210,5 @@
     origin_rpy="0.0 0.0 0.0"
     meshfile="package://rjje_arm/meshes/motor_and_frame.stl"
-    meshscale="0.1 0.1 0.1"
+    meshscale="${scale_factor} ${scale_factor} ${scale_factor}"
     mass="1.57633"
     ixx="0.13235" ixy="0" ixz="0"
@@ -249,5 +250,5 @@
     origin_rpy="0.0 0.0 0.0"
     meshfile="package://rjje_arm/meshes/gripper_finger.stl"
-    meshscale="0.1 0.1 0.1"
+    meshscale="${scale_factor} ${scale_factor} ${scale_factor}"
     mass="1.57633"
     ixx="0.13235" ixy="0" ixz="0"
@@ -269,5 +270,5 @@
     origin_rpy="0.0 0.0 0.0"
     meshfile="package://rjje_arm/meshes/gripper_finger.stl"
-    meshscale="0.1 0.1 0.1"
+    meshscale="${scale_factor} ${scale_factor} ${scale_factor}"
     mass="1.57633"
     ixx="0.13235" ixy="0" ixz="0"

File: RJJE_Arm/rjje_arm_ws/src/rjje_arm/urdf/rjje_arm.xacro.urdf (robot description, URDF)
Before this commit: robot rjje_arm, 15 links, 14 joints
Links:
- link base_link: geometry collision mesh filename=package://rjje_arm/meshes/base.stl scale=0.01 0.01 0.01; visual mesh filename=package://rjje_arm/meshes/base.stl scale=0.01 0.01 0.01
- link bracket_1: geometry collision mesh filename=package://rjje_arm/meshes/thin_bracket.stl scale=0.01 0.01 0.01; visual mesh filename=package://rjje_arm/meshes/thin_bracket.stl scale=0.01 0.01 0.01
- link bracket_2_1: geometry collision mesh filename=package://rjje_arm/meshes/thin_bracket.stl scale=0.01 0.01 0.01; visual mesh filename=package://rjje_arm/meshes/thin_bracket.stl scale=0.01 0.01 0.01
- link bracket_2_2: geometry collision mesh filename=package://rjje_arm/meshes/thin_bracket.stl scale=0.01 0.01 0.01; visual mesh filename=package://rjje_arm/meshes/thin_bracket.stl scale=0.01 0.01 0.01
- link bracket_3_1: geometry collision cylinder length=0.015 radius=0.005; visual cylinder length=0.015 radius=0.005
- link bracket_3_2: geometry collision mesh filename=package://rjje_arm/meshes/thin_bracket.stl scale=0.01 0.01 0.01; visual mesh filename=package://rjje_arm/meshes/thin_bracket.stl scale=0.01 0.01 0.01
- link left_gripper: geometry collision mesh filename=package://rjje_arm/meshes/gripper_finger.stl scale=0.01 0.01 0.01; visual mesh filename=package://rjje_arm/meshes/gripper_finger.stl scale=0.01 0.01 0.01
- link link1: geometry collision mesh filename=package://rjje_arm/meshes/motor_and_frame.stl scale=0.01 0.01 0.01; visual mesh filename=package://rjje_arm/meshes/motor_and_frame.stl scale=0.01 0.01 0.01
- link link_2: geometry collision mesh filename=package://rjje_arm/meshes/motor_and_frame.stl scale=0.01 0.01 0.01; visual mesh filename=package://rjje_arm/meshes/motor_and_frame.stl scale=0.01 0.01 0.01
- link link_3: geometry collision mesh filename=package://rjje_arm/meshes/motor_and_frame.stl scale=0.01 0.01 0.01; visual mesh filename=package://rjje_arm/meshes/motor_and_frame.stl scale=0.01 0.01 0.01
- link link_4: geometry collision mesh filename=package://rjje_arm/meshes/motor_and_frame.stl scale=0.01 0.01 0.01; visual mesh filename=package://rjje_arm/meshes/motor_and_frame.stl scale=0.01 0.01 0.01
- link link_5: geometry collision mesh filename=package://rjje_arm/meshes/motor_and_frame.stl scale=0.01 0.01 0.01; visual mesh filename=package://rjje_arm/meshes/motor_and_frame.stl scale=0.01 0.01 0.01
- link right_gripper: geometry collision mesh filename=package://rjje_arm/meshes/gripper_finger.stl scale=0.01 0.01 0.01; visual mesh filename=package://rjje_arm/meshes/gripper_finger.stl scale=0.01 0.01 0.01
Joints:
- joint base_link_link1: origin xyz=0.34500000000000003 0.42000000000000004 0.4 rpy=0 0 0 -> xyz=0.0345 0.042 0.04 rpy=0 0 0
- joint bracket_1_link_2: origin xyz=0.22000000000000003 0.0 0.13999999999999999 rpy=1.57 0.0 -1.57 -> xyz=0.022000000000000002 0.0 0.013999999999999999 rpy=1.57 0.0 -1.57
- joint bracket_2_1_bracket_2_2: origin xyz=0.0 1.05 0.0 rpy=0.0 0.0 3.14 -> xyz=0.0 0.105 0.0 rpy=0.0 0.0 3.14
- joint bracket_2_2_link_3: origin xyz=0.0 0.0 -0.53 rpy=0.0 0.0 3.14 -> xyz=0.0 0.0 -0.053 rpy=0.0 0.0 3.14
- joint bracket_3_1_bracket_3_2: origin xyz=-0.265 0.0 0.675 rpy=-1.57 0.0 1.57 -> xyz=-0.0265 0.0 0.0675 rpy=-1.57 0.0 1.57
- joint bracket_3_2_link_4: origin xyz=0.0 0.0 -0.53 rpy=0.0 0.0 -1.57 -> xyz=0.0 0.0 -0.053 rpy=0.0 0.0 -1.57
- joint link1_bracket_1: origin xyz=0.0 0.0 0.53 rpy=0 0 0 -> xyz=0.0 0.0 0.053 rpy=0 0 0
- joint link_2_bracket_2_1: origin xyz=0.0 0.0 0.53 rpy=0.0 0.0 0.0 -> xyz=0.0 0.0 0.053 rpy=0.0 0.0 0.0
- joint link_3_bracket_3_1: origin xyz=0.4 0.0 0.2 rpy=0.0 1.57 0.0 -> xyz=0.04 0.0 0.02 rpy=0.0 1.57 0.0
- joint link_4_link_5: origin xyz=0.0 0.24 0.22000000000000003 rpy=0.0 1.57 0.0 -> xyz=0.0 0.024 0.022000000000000002 rpy=0.0 1.57 0.0
- joint link_5_link_6: origin xyz=0.0 0.0 0.52 rpy=0.0 0.0 0.0 -> xyz=0.0 0.0 0.052000000000000005 rpy=0.0 0.0 0.0
- joint link_6_left_gripper: origin xyz=-0.16000000000000003 0.0 0.16000000000000003 rpy=1.57 0.0 0.0 -> xyz=-0.016 0.0 0.016 rpy=1.57 0.0 0.0
- joint link_6_right_gripper: origin xyz=0.16000000000000003 0.0 0.16000000000000003 rpy=1.57 0.0 0.0 -> xyz=0.016 0.0 0.016 rpy=1.57 0.0 0.0
