Commit message: lots of modifications: going to implement soft-real time independent gripper and arm control

File: RJJE_Arm/rjje_arm_ws/src/rjje_arm/urdf/rjje_arm.xacro (robot description, xacro)
@@ -206,22 +206,22 @@
   <xacro:m_joint type="revolute"
     axis_xyz="0 0 1"
+    origin_xyz="0.0 0.0 5.2" origin_rpy="0.0 0.0 0.0"
+    parent="link_5" child="link_6"
+    limit_e="1000" limit_l="-1.57" limit_u="1.57" limit_v="1.5" />
+  <xacro:m_link_mesh
+    name="left_gripper"
+    origin_xyz="0.0 0.0 0.0"
+    origin_rpy="0.0 0.0 0.0"
+    meshfile="package://rjje_arm/meshes/left_gripper.stl"
+    meshscale="1 1 1"
+    mass="157.633"
+    ixx="13.235" ixy="0" ixz="0"
+    iyy="13.235" iyz="0"
+    izz="9.655"
+    color="yellow"
+    />
+  <xacro:m_joint type="revolute"
+    axis_xyz="0 1 0"
     origin_xyz="0.0 0.0 0.0" origin_rpy="0.0 0.0 0.0"
-    parent="link_5" child="link_6"
-    limit_e="1000" limit_l="-1.57" limit_u="1.57" limit_v="1.5" />
-  <xacro:m_link_mesh
-    name="left_gripper"
-    origin_xyz="0.0 0.0 0.0"
-    origin_rpy="0.0 0.0 0.0"
-    meshfile="package://rjje_arm/meshes/left_gripper.stl"
-    meshscale="1 1 1"
-    mass="157.633"
-    ixx="13.235" ixy="0" ixz="0"
-    iyy="13.235" iyz="0"
-    izz="9.655"
-    color="yellow"
-    />
-  <xacro:m_joint type="revolute"
-    axis_xyz="0 1 0"
-    origin_xyz="0.0 0.0 5.2" origin_rpy="0.0 0.0 0.0"
     parent="link_6" child="left_gripper"
     limit_e="1000" limit_l="-0.61" limit_u="0.0" limit_v="1.5" />
@@ -243,5 +243,5 @@
     type="revolute"
     axis_xyz="0 1 0"
-    origin_xyz="0.0 0.0 5.2" origin_rpy="0.0 0.0 0.0"
+    origin_xyz="0.0 0.0 0.0" origin_rpy="0.0 0.0 0.0"
     parent="link_6" child="right_gripper"
     limit_e="1000" limit_l="0.61" limit_u="0.0" limit_v="1.5"

File: RJJE_Arm/rjje_arm_ws/src/rjje_arm/urdf/rjje_arm.xacro.urdf (robot description, URDF)
Before this commit: robot rjje_arm, 15 links, 14 joints
Joints:
- joint link_5_link_6: origin xyz=0.0 0.0 0.0 rpy=0.0 0.0 0.0 -> xyz=0.0 0.0 5.2 rpy=0.0 0.0 0.0
- joint link_6_left_gripper: origin xyz=0.0 0.0 5.2 rpy=0.0 0.0 0.0 -> xyz=0.0 0.0 0.0 rpy=0.0 0.0 0.0
- joint link_6_right_gripper: origin xyz=0.0 0.0 5.2 rpy=0.0 0.0 0.0 -> xyz=0.0 0.0 0.0 rpy=0.0 0.0 0.0

Commit message: definitions

File: RJJE_Arm/rjje_arm_ws/src/rjje_arm/urdf/rjje_arm.xacro (robot description, xacro)
@@ -3,4 +3,6 @@
   <xacro:include filename="$(find rjje_arm)/urdf/definitions.xacro" />
   <!-- Instances -->
+  <!-- Gazebo colors: https://github.com/osrf/gazebo/blob/master/media/materials/scripts/gazebo.material -->
+  <!-- rosrun xacro xacro - -inorder -o model.urdf model.urdf.xacro -->
   <link name="world">
   </link>
@@ -18,5 +20,5 @@
     />
   <gazebo reference="base_link">
-    <material>Gazebo/Yellow</material>
+    <material>Gazebo/RedGlow</material>
   </gazebo>
   <xacro:m_joint type="fixed"
@@ -37,4 +39,7 @@
     color="dark_green"
     />
+  <gazebo reference="link1">
+    <material>Gazebo/RedGlow</material>
+  </gazebo>
   <xacro:m_joint type="fixed"
     axis_xyz="0 0 1"
@@ -54,4 +59,7 @@
     color="blue"
     />
+  <gazebo reference="bracket_1">
+    <material>Gazebo/RedGlow</material>
+  </gazebo>
   <xacro:m_joint type="revolute"
     axis_xyz="0 0 1"
@@ -71,4 +79,7 @@
     color="dark_green"
     />
+  <gazebo reference="link_2">
+    <material>Gazebo/RedGlow</material>
+  </gazebo>
   <xacro:m_joint type="fixed"
     axis_xyz="0 0 1"
@@ -88,4 +99,7 @@
     color="blue"
     />
+  <gazebo reference="bracket_2_1">
+    <material>Gazebo/RedGlow</material>
+  </gazebo>
   <xacro:m_joint type="revolute"
     axis_xyz="0 0 1"
@@ -105,4 +119,7 @@
     color="blue"
     />
+  <gazebo reference="bracket_2_2">
+    <material>Gazebo/RedGlow</material>
+  </gazebo>
   <xacro:m_joint type="fixed"
     axis_xyz="0 0 1"
@@ -122,4 +139,7 @@
     color="dark_green"
     />
+  <gazebo reference="link_3">
+    <material>Gazebo/RedGlow</material>
+  </gazebo>
   <xacro:m_joint type="revolute"
     axis_xyz="0 0 1"
@@ -130,5 +150,5 @@
   <xacro:m_fake_link
     name="bracket_3_1"
-    color="pink"
+    color="Yellow"
     origin_xyz="0.0 0.0 0.75"
     origin_rpy="0.0 0.0 0.0"
@@ -136,4 +156,7 @@
     radius="0.5"
     />
+  <gazebo reference="bracket_3_1">
+    <material>Gazebo/RedGlow</material>
+  </gazebo>
   <xacro:m_joint type="fixed"
     axis_xyz="0 0 1"
@@ -153,4 +176,7 @@
     color="blue"
     />
+  <gazebo reference="bracket_3_2">
+    <material>Gazebo/RedGlow</material>
+  </gazebo>
   <xacro:m_joint type="fixed"
     axis_xyz="0 0 1"
@@ -170,4 +196,7 @@
     color="dark_green"
     />
+  <gazebo reference="link_4">
+    <material>Gazebo/RedGlow</material>
+  </gazebo>
   <xacro:m_joint type="revolute"
     axis_xyz="0 0 1"
@@ -187,4 +216,7 @@
     color="dark_green"
     />
+  <gazebo reference="link_5">
+    <material>Gazebo/RedGlow</material>
+  </gazebo>
   <xacro:m_joint type="fixed"
     axis_xyz="0 0 1"
@@ -204,4 +236,7 @@
     color="dark_green"
     />
+  <gazebo reference="link_6">
+    <material>Gazebo/RedGlow</material>
+  </gazebo>
   <xacro:m_joint type="revolute"
     axis_xyz="0 0 1"
@@ -221,4 +256,7 @@
     color="yellow"
     />
+  <gazebo reference="left_gripper">
+    <material>Gazebo/RedGlow</material>
+  </gazebo>
   <xacro:m_joint type="revolute"
     axis_xyz="0 1 0"
@@ -238,4 +276,7 @@
     color="yellow"
     />
+  <gazebo reference="right_gripper">
+    <material>Gazebo/RedGlow</material>
+  </gazebo>
   <xacro:m_mimic_joint
     joint_parent="link_6"

Commit message: lots of changes to rjje arm: gazebo, esp32, servo control

File: RJJE_Arm/rjje_arm_ws/src/rjje_arm/urdf/rjje_arm.xacro (robot description, xacro)
@@ -20,5 +20,5 @@
     />
   <gazebo reference="base_link">
-    <material>Gazebo/RedGlow</material>
+    <material>Gazebo/Purple</material>
   </gazebo>
   <xacro:m_joint type="fixed"
@@ -40,5 +40,5 @@
     />
   <gazebo reference="link1">
-    <material>Gazebo/RedGlow</material>
+    <material>Gazebo/Turquoise</material>
   </gazebo>
   <xacro:m_joint type="fixed"
@@ -60,5 +60,5 @@
     />
   <gazebo reference="bracket_1">
-    <material>Gazebo/RedGlow</material>
+    <material>Gazebo/PurpleGlow</material>
   </gazebo>
   <xacro:m_joint type="revolute"
@@ -80,5 +80,5 @@
     />
   <gazebo reference="link_2">
-    <material>Gazebo/RedGlow</material>
+    <material>Gazebo/Wood</material>
   </gazebo>
   <xacro:m_joint type="fixed"
@@ -100,5 +100,5 @@
     />
   <gazebo reference="bracket_2_1">
-    <material>Gazebo/RedGlow</material>
+    <material>Gazebo/PurpleGlow</material>
   </gazebo>
   <xacro:m_joint type="revolute"
@@ -120,5 +120,5 @@
     />
   <gazebo reference="bracket_2_2">
-    <material>Gazebo/RedGlow</material>
+    <material>Gazebo/PurpleGlow</material>
   </gazebo>
   <xacro:m_joint type="fixed"
@@ -140,5 +140,5 @@
     />
   <gazebo reference="link_3">
-    <material>Gazebo/RedGlow</material>
+    <material>Gazebo/Indigo</material>
   </gazebo>
   <xacro:m_joint type="revolute"
@@ -157,5 +157,5 @@
     />
   <gazebo reference="bracket_3_1">
-    <material>Gazebo/RedGlow</material>
+    <material>Gazebo/PurpleGlow</material>
   </gazebo>
   <xacro:m_joint type="fixed"
@@ -177,5 +177,5 @@
     />
   <gazebo reference="bracket_3_2">
-    <material>Gazebo/RedGlow</material>
+    <material>Gazebo/PurpleGlow</material>
   </gazebo>
   <xacro:m_joint type="fixed"
@@ -197,5 +197,5 @@
     />
   <gazebo reference="link_4">
-    <material>Gazebo/RedGlow</material>
+    <material>Gazebo/Indigo</material>
   </gazebo>
   <xacro:m_joint type="revolute"
@@ -217,5 +217,5 @@
     />
   <gazebo reference="link_5">
-    <material>Gazebo/RedGlow</material>
+    <material>Gazebo/PurpleGlow</material>
   </gazebo>
   <xacro:m_joint type="fixed"
@@ -237,5 +237,5 @@
     />
   <gazebo reference="link_6">
-    <material>Gazebo/RedGlow</material>
+    <material>Gazebo/Orange</material>
   </gazebo>
   <xacro:m_joint type="revolute"
@@ -257,5 +257,5 @@
     />
   <gazebo reference="left_gripper">
-    <material>Gazebo/RedGlow</material>
+    <material>Gazebo/Gold</material>
   </gazebo>
   <xacro:m_joint type="revolute"
@@ -277,5 +277,5 @@
     />
   <gazebo reference="right_gripper">
-    <material>Gazebo/RedGlow</material>
+    <material>Gazebo/Gold</material>
   </gazebo>
   <xacro:m_mimic_joint

Commit message: added gripper stl

File: RJJE_Arm/rjje_arm_ws/src/rjje_arm/urdf/rjje_arm.xacro (robot description, xacro)
@@ -248,5 +248,5 @@
     origin_xyz="0.0 0.0 0.0"
     origin_rpy="0.0 0.0 0.0"
-    meshfile="package://rjje_arm/meshes/left_gripper.stl"
+    meshfile="package://rjje_arm/meshes/gripper_finger.stl"
     meshscale="1 1 1"
     mass="157.633"
@@ -260,13 +260,13 @@
   </gazebo>
   <xacro:m_joint type="revolute"
-    axis_xyz="0 1 0"
-    origin_xyz="0.0 0.0 0.0" origin_rpy="0.0 0.0 0.0"
+    axis_xyz="0 0 1"
+    origin_xyz="-1.6 0.0 1.6" origin_rpy="1.57 0.0 0.0"
     parent="link_6" child="left_gripper"
-    limit_e="1000" limit_l="-0.61" limit_u="0.0" limit_v="1.5" />
+    limit_e="1000" limit_l="0.0" limit_u="0.61" limit_v="1.5" />
   <xacro:m_link_mesh
     name="right_gripper"
     origin_xyz="0.0 0.0 0.0"
     origin_rpy="0.0 0.0 0.0"
-    meshfile="package://rjje_arm/meshes/right_gripper.stl"
+    meshfile="package://rjje_arm/meshes/gripper_finger.stl"
     meshscale="1 1 1"
     mass="157.633"
@@ -283,8 +283,8 @@
     joint_child="left_gripper"
     type="revolute"
-    axis_xyz="0 1 0"
-    origin_xyz="0.0 0.0 0.0" origin_rpy="0.0 0.0 0.0"
+    axis_xyz="0 0 1"
+    origin_xyz="1.6 0.0 1.6" origin_rpy="1.57 0.0 0.0"
     parent="link_6" child="right_gripper"
-    limit_e="1000" limit_l="0.61" limit_u="0.0" limit_v="1.5"
+    limit_e="1000" limit_l="-0.61" limit_u="0.0" limit_v="1.5"
     multiplier="-1"
     offset="0"

File: RJJE_Arm/rjje_arm_ws/src/rjje_arm/urdf/rjje_arm.xacro.urdf (robot description, URDF)
Before this commit: robot rjje_arm, 15 links, 14 joints
Links:
- link left_gripper: geometry collision mesh filename=package://rjje_arm/meshes/gripper_finger.stl scale=1 1 1; visual mesh filename=package://rjje_arm/meshes/gripper_finger.stl scale=1 1 1
- link right_gripper: geometry collision mesh filename=package://rjje_arm/meshes/gripper_finger.stl scale=1 1 1; visual mesh filename=package://rjje_arm/meshes/gripper_finger.stl scale=1 1 1
Joints:
- joint link_6_left_gripper: axis 0 1 0 -> 0 0 1; limit lower=-0.61 upper=0.0 effort=1000 velocity=1.5 -> lower=0.0 upper=0.61 effort=1000 velocity=1.5; origin xyz=0.0 0.0 0.0 rpy=0.0 0.0 0.0 -> xyz=-1.6 0.0 1.6 rpy=1.57 0.0 0.0
- joint link_6_right_gripper: axis 0 1 0 -> 0 0 1; limit lower=0.61 upper=0.0 effort=1000 velocity=1.5 -> lower=-0.61 upper=0.0 effort=1000 velocity=1.5; origin xyz=0.0 0.0 0.0 rpy=0.0 0.0 0.0 -> xyz=1.6 0.0 1.6 rpy=1.57 0.0 0.0

Commit message: mass

File: RJJE_Arm/rjje_arm_ws/src/rjje_arm/urdf/rjje_arm.xacro (robot description, xacro)
@@ -13,8 +13,8 @@
     meshfile="package://rjje_arm/meshes/base.stl"
     meshscale="1 1 1"
-    mass="157.633"
-    ixx="13.235" ixy="0" ixz="0"
-    iyy="13.235" iyz="0"
-    izz="9.655"
+    mass="1.57633"
+    ixx="0.13235" ixy="0" ixz="0"
+    iyy="0.13235" iyz="0"
+    izz="0.09655"
     color="yellow"
     />
@@ -33,8 +33,8 @@
     meshfile="package://rjje_arm/meshes/motor_and_frame.stl"
     meshscale="1 1 1"
-    mass="157.633"
-    ixx="13.235" ixy="0" ixz="0"
-    iyy="13.235" iyz="0"
-    izz="9.655"
+    mass="1.57633"
+    ixx="0.13235" ixy="0" ixz="0"
+    iyy="0.13235" iyz="0"
+    izz="0.09655"
     color="dark_green"
     />
@@ -53,8 +53,8 @@
     meshfile="package://rjje_arm/meshes/thin_bracket.stl"
     meshscale="1 1 1"
-    mass="157.633"
-    ixx="13.235" ixy="0" ixz="0"
-    iyy="13.235" iyz="0"
-    izz="9.655"
+    mass="1.57633"
+    ixx="0.13235" ixy="0" ixz="0"
+    iyy="0.13235" iyz="0"
+    izz="0.09655"
     color="blue"
     />
@@ -73,8 +73,8 @@
     meshfile="package://rjje_arm/meshes/motor_and_frame.stl"
     meshscale="1 1 1"
-    mass="157.633"
-    ixx="13.235" ixy="0" ixz="0"
-    iyy="13.235" iyz="0"
-    izz="9.655"
+    mass="1.57633"
+    ixx="0.13235" ixy="0" ixz="0"
+    iyy="0.13235" iyz="0"
+    izz="0.09655"
     color="dark_green"
     />
@@ -93,8 +93,8 @@
     meshfile="package://rjje_arm/meshes/thin_bracket.stl"
     meshscale="1 1 1"
-    mass="157.633"
-    ixx="13.235" ixy="0" ixz="0"
-    iyy="13.235" iyz="0"
-    izz="9.655"
+    mass="1.57633"
+    ixx="0.13235" ixy="0" ixz="0"
+    iyy="0.13235" iyz="0"
+    izz="0.09655"
     color="blue"
     />
@@ -113,8 +113,8 @@
     meshfile="package://rjje_arm/meshes/thin_bracket.stl"
     meshscale="1 1 1"
-    mass="157.633"
-    ixx="13.235" ixy="0" ixz="0"
-    iyy="13.235" iyz="0"
-    izz="9.655"
+    mass="1.57633"
+    ixx="0.13235" ixy="0" ixz="0"
+    iyy="0.13235" iyz="0"
+    izz="0.09655"
     color="blue"
     />
@@ -133,8 +133,8 @@
     meshfile="package://rjje_arm/meshes/motor_and_frame.stl"
     meshscale="1 1 1"
-    mass="157.633"
-    ixx="13.235" ixy="0" ixz="0"
-    iyy="13.235" iyz="0"
-    izz="9.655"
+    mass="1.57633"
+    ixx="0.13235" ixy="0" ixz="0"
+    iyy="0.13235" iyz="0"
+    izz="0.09655"
     color="dark_green"
     />
@@ -170,8 +170,8 @@
     meshfile="package://rjje_arm/meshes/thin_bracket.stl"
     meshscale="1 1 1"
-    mass="157.633"
-    ixx="13.235" ixy="0" ixz="0"
-    iyy="13.235" iyz="0"
-    izz="9.655"
+    mass="1.57633"
+    ixx="0.13235" ixy="0" ixz="0"
+    iyy="0.13235" iyz="0"
+    izz="0.09655"
     color="blue"
     />
@@ -190,8 +190,8 @@
     meshfile="package://rjje_arm/meshes/motor_and_frame.stl"
     meshscale="1 1 1"
-    mass="157.633"
-    ixx="13.235" ixy="0" ixz="0"
-    iyy="13.235" iyz="0"
-    izz="9.655"
+    mass="1.57633"
+    ixx="0.13235" ixy="0" ixz="0"
+    iyy="0.13235" iyz="0"
+    izz="0.09655"
     color="dark_green"
     />
@@ -210,8 +210,8 @@
     meshfile="package://rjje_arm/meshes/motor_and_frame.stl"
     meshscale="1 1 1"
-    mass="157.633"
-    ixx="13.235" ixy="0" ixz="0"
-    iyy="13.235" iyz="0"
-    izz="9.655"
+    mass="1.57633"
+    ixx="0.13235" ixy="0" ixz="0"
+    iyy="0.13235" iyz="0"
+    izz="0.09655"
     color="dark_green"
     />
@@ -230,8 +230,8 @@
     meshfile="package://rjje_arm/meshes/motor_and_frame.stl"
     meshscale="0 0 0"
-    mass="157.633"
-    ixx="13.235" ixy="0" ixz="0"
-    iyy="13.235" iyz="0"
-    izz="9.655"
+    mass="1.57633"
+    ixx="0.13235" ixy="0" ixz="0"
+    iyy="0.13235" iyz="0"
+    izz="0.09655"
     color="dark_green"
     />
@@ -250,8 +250,8 @@
     meshfile="package://rjje_arm/meshes/gripper_finger.stl"
     meshscale="1 1 1"
-    mass="157.633"
-    ixx="13.235" ixy="0" ixz="0"
-    iyy="13.235" iyz="0"
-    izz="9.655"
+    mass="1.57633"
+    ixx="0.13235" ixy="0" ixz="0"
+    iyy="0.13235" iyz="0"
+    izz="0.09655"
     color="yellow"
     />
@@ -270,8 +270,8 @@
     meshfile="package://rjje_arm/meshes/gripper_finger.stl"
     meshscale="1 1 1"
-    mass="157.633"
-    ixx="13.235" ixy="0" ixz="0"
-    iyy="13.235" iyz="0"
-    izz="9.655"
+    mass="1.57633"
+    ixx="0.13235" ixy="0" ixz="0"
+    iyy="0.13235" iyz="0"
+    izz="0.09655"
     color="yellow"
     />

File: RJJE_Arm/rjje_arm_ws/src/rjje_arm/urdf/rjje_arm.xacro.urdf (robot description, URDF)
Before this commit: robot rjje_arm, 15 links, 14 joints
Links:
- link base_link: mass 157.633 -> 1.57633
- link bracket_1: mass 157.633 -> 1.57633
- link bracket_2_1: mass 157.633 -> 1.57633
- link bracket_2_2: mass 157.633 -> 1.57633
- link bracket_3_2: mass 157.633 -> 1.57633
- link left_gripper: mass 157.633 -> 1.57633
- link link1: mass 157.633 -> 1.57633
- link link_2: mass 157.633 -> 1.57633
- link link_3: mass 157.633 -> 1.57633
- link link_4: mass 157.633 -> 1.57633
- link link_5: mass 157.633 -> 1.57633
- link link_6: mass 157.633 -> 1.57633
- link right_gripper: mass 157.633 -> 1.57633
