Commit message: ros control works!

File: RJJE_Arm/rjje_arm_ws/src/rjje_arm/urdf/rjje_arm.xacro (robot description, xacro)
@@ -28,5 +28,5 @@
     origin_rpy="0 0 0" origin_xyz="0 0 0.0"
     parent="world" child="base_link"
-    limit_e="1000" limit_l="0" limit_u="0.5" limit_v="0.5" />
+    limit_e="50" limit_l="0" limit_u="0.5" limit_v="0.5" />
   <xacro:m_link_mesh
     name="link1"
@@ -48,5 +48,5 @@
     origin_rpy="0 0 0" origin_xyz="3.45 4.2 4.0"
     parent="base_link" child="link1"
-    limit_e="1000" limit_l="0" limit_u="0.5" limit_v="0.5" />
+    limit_e="50" limit_l="0" limit_u="0.5" limit_v="0.5" />
   <xacro:m_link_mesh
     name="bracket_1"
@@ -68,5 +68,5 @@
     origin_rpy="0 0 0" origin_xyz="0 0 5.3"
     parent="link1" child="bracket_1"
-    limit_e="1000" limit_l="-1.57" limit_u="1.57" limit_v="1.5" />
+    limit_e="50" limit_l="-1.57" limit_u="1.57" limit_v="1.5" />
   <xacro:m_link_mesh
     name="link_2"
@@ -88,5 +88,5 @@
     origin_xyz="2.2 0.0 1.4" origin_rpy="1.57 0.0 -1.57"
     parent="bracket_1" child="link_2"
-    limit_e="1000" limit_l="-1.57" limit_u="1.57" limit_v="0.5" />
+    limit_e="50" limit_l="-1.57" limit_u="1.57" limit_v="0.5" />
   <xacro:m_link_mesh
     name="bracket_2_1"
@@ -108,5 +108,5 @@
     origin_xyz="0.0 0.0 5.3" origin_rpy="0.0 0.0 0.0"
     parent="link_2" child="bracket_2_1"
-    limit_e="1000" limit_l="-1.57" limit_u="1.57" limit_v="1.5" />
+    limit_e="50" limit_l="-1.57" limit_u="1.57" limit_v="1.5" />
   <xacro:m_link_mesh
     name="bracket_2_2"
@@ -128,5 +128,5 @@
     origin_xyz="0.0 10.5 0.0" origin_rpy="0.0 0.0 3.14"
     parent="bracket_2_1" child="bracket_2_2"
-    limit_e="1000" limit_l="-1.57" limit_u="1.57" limit_v="0.5" />
+    limit_e="50" limit_l="-1.57" limit_u="1.57" limit_v="0.5" />
   <xacro:m_link_mesh
     name="link_3"
@@ -148,5 +148,5 @@
     origin_xyz="0.0 0.0 -5.3" origin_rpy="0.0 0.0 3.14"
     parent="bracket_2_2" child="link_3"
-    limit_e="1000" limit_l="-1.57" limit_u="1.57" limit_v="1.5" />
+    limit_e="50" limit_l="-1.57" limit_u="1.57" limit_v="1.5" />
   <!-- This is a "fake" link that represents attachment to link 3 -->
   <xacro:m_fake_link
@@ -165,5 +165,5 @@
     origin_xyz="4.0 0.0 2.0" origin_rpy="0.0 1.57 0.0"
     parent="link_3" child="bracket_3_1"
-    limit_e="1000" limit_l="-1.57" limit_u="1.57" limit_v="0.5" />
+    limit_e="50" limit_l="-1.57" limit_u="1.57" limit_v="0.5" />
   <xacro:m_link_mesh
     name="bracket_3_2"
@@ -185,5 +185,5 @@
     origin_xyz="-2.65 0.0 6.75" origin_rpy="-1.57 0.0 1.57"
     parent="bracket_3_1" child="bracket_3_2"
-    limit_e="1000" limit_l="-1.57" limit_u="1.57" limit_v="0.5" />
+    limit_e="50" limit_l="-1.57" limit_u="1.57" limit_v="0.5" />
   <xacro:m_link_mesh
     name="link_4"
@@ -205,5 +205,5 @@
     origin_xyz="0.0 0.0 -5.3" origin_rpy="0.0 0.0 -1.57"
     parent="bracket_3_2" child="link_4"
-    limit_e="1000" limit_l="-1.57" limit_u="0.43" limit_v="1.5" />
+    limit_e="50" limit_l="-1.57" limit_u="0.43" limit_v="1.5" />
   <xacro:m_link_mesh
     name="link_5"
@@ -225,5 +225,5 @@
     origin_xyz="0.0 2.4 2.2" origin_rpy="0.0 1.57 0.0"
     parent="link_4" child="link_5"
-    limit_e="1000" limit_l="-1.57" limit_u="1.57" limit_v="0.5" />
+    limit_e="50" limit_l="-1.57" limit_u="1.57" limit_v="0.5" />
   <xacro:m_link_mesh
     name="link_6"
@@ -245,5 +245,5 @@
     origin_xyz="0.0 0.0 5.2" origin_rpy="0.0 0.0 0.0"
     parent="link_5" child="link_6"
-    limit_e="1000" limit_l="-1.57" limit_u="1.57" limit_v="1.5" />
+    limit_e="50" limit_l="-1.57" limit_u="1.57" limit_v="1.5" />
   <xacro:m_link_mesh
     name="left_gripper"
@@ -265,5 +265,5 @@
     origin_xyz="-1.6 0.0 1.6" origin_rpy="1.57 0.0 0.0"
     parent="link_6" child="left_gripper"
-    limit_e="1000" limit_l="0.0" limit_u="0.61" limit_v="1.5" />
+    limit_e="50" limit_l="0.0" limit_u="0.61" limit_v="1.5" />
   <xacro:m_link_mesh
     name="right_gripper"
@@ -288,5 +288,5 @@
     origin_xyz="1.6 0.0 1.6" origin_rpy="1.57 0.0 0.0"
     parent="link_6" child="right_gripper"
-    limit_e="1000" limit_l="-0.61" limit_u="0.0" limit_v="1.5"
+    limit_e="50" limit_l="-0.61" limit_u="0.0" limit_v="1.5"
     multiplier="-1"
     offset="0"

File: RJJE_Arm/rjje_arm_ws/src/rjje_arm/urdf/rjje_arm.xacro.urdf (robot description, URDF)
Before this commit: robot rjje_arm, 15 links, 14 joints
Links:
- link base_link: mass 1.57633 -> 0.0157633
- link bracket_1: mass 1.57633 -> 0.0157633
- link bracket_2_1: mass 1.57633 -> 0.0157633
- link bracket_2_2: mass 1.57633 -> 0.0157633
- link bracket_3_2: mass 1.57633 -> 0.0157633
- link left_gripper: mass 1.57633 -> 0.0157633
- link link1: mass 1.57633 -> 0.0157633
- link link_2: mass 1.57633 -> 0.0157633
- link link_3: mass 1.57633 -> 0.0157633
- link link_4: mass 1.57633 -> 0.0157633
- link link_5: mass 1.57633 -> 0.0157633
- link link_6: mass 1.57633 -> 0.0157633
- link right_gripper: mass 1.57633 -> 0.0157633
Joints:
- joint base_link_link1: limit lower=0 upper=0.5 effort=1000 velocity=0.5 -> lower=0 upper=0.5 effort=50 velocity=0.5
- joint bracket_1_link_2: limit lower=-1.57 upper=1.57 effort=1000 velocity=0.5 -> lower=-1.57 upper=1.57 effort=50 velocity=0.5
- joint bracket_2_1_bracket_2_2: limit lower=-1.57 upper=1.57 effort=1000 velocity=0.5 -> lower=-1.57 upper=1.57 effort=50 velocity=0.5
- joint bracket_2_2_link_3: limit lower=-1.57 upper=1.57 effort=1000 velocity=1.5 -> lower=-1.57 upper=1.57 effort=50 velocity=1.5
- joint bracket_3_1_bracket_3_2: limit lower=-1.57 upper=1.57 effort=1000 velocity=0.5 -> lower=-1.57 upper=1.57 effort=50 velocity=0.5
- joint bracket_3_2_link_4: limit lower=-1.57 upper=0.43 effort=1000 velocity=1.5 -> lower=-1.57 upper=0.43 effort=50 velocity=1.5
- joint link1_bracket_1: limit lower=-1.57 upper=1.57 effort=1000 velocity=1.5 -> lower=-1.57 upper=1.57 effort=50 velocity=1.5
- joint link_2_bracket_2_1: limit lower=-1.57 upper=1.57 effort=1000 velocity=1.5 -> lower=-1.57 upper=1.57 effort=50 velocity=1.5
- joint link_3_bracket_3_1: limit lower=-1.57 upper=1.57 effort=1000 velocity=0.5 -> lower=-1.57 upper=1.57 effort=50 velocity=0.5
- joint link_4_link_5: limit lower=-1.57 upper=1.57 effort=1000 velocity=0.5 -> lower=-1.57 upper=1.57 effort=50 velocity=0.5
- joint link_5_link_6: limit lower=-1.57 upper=1.57 effort=1000 velocity=1.5 -> lower=-1.57 upper=1.57 effort=50 velocity=1.5
- joint link_6_left_gripper: limit lower=0.0 upper=0.61 effort=1000 velocity=1.5 -> lower=0.0 upper=0.61 effort=50 velocity=1.5
- joint link_6_right_gripper: limit lower=-0.61 upper=0.0 effort=1000 velocity=1.5 -> lower=-0.61 upper=0.0 effort=50 velocity=1.5
- joint world_base_link: limit lower=0 upper=0.5 effort=1000 velocity=0.5 -> lower=0 upper=0.5 effort=50 velocity=0.5

File: RJJE_Arm/rjje_arm_ws/src/rjje_arm/urdf/ros_control.xacro (robot description, xacro)
@@ -1,13 +1,25 @@
 <?xml version="1.0"?>
-<robot name="ros_control" xmlns:xacro="http://www.ros.org/wiki/xacro">
-  <transmission name="tran1">
-    <type>transmission_interface/SimpleTransmission</type>
-    <joint name="link1_bracket_1">
-      <hardwareInterface>PositionJointInterface</hardwareInterface>
-    </joint>
-    <actuator name="motor1">
-      <hardwareInterface>PositionJointInterface</hardwareInterface>
-      <mechanicalReduction>1</mechanicalReduction>
-    </actuator>
-  </transmission>
+    <robot name="definitions" xmlns:xacro="http://www.ros.org/wiki/xacro">
+        <xacro:macro name="m_transmission" params="index joint_name">
+            <transmission name="tran_${index}">
+            <type>transmission_interface/SimpleTransmission</type>
+            <joint name="${joint_name}">
+                <hardwareInterface>EffortJointInterface</hardwareInterface>
+            </joint>
+            <actuator name="motor_${index}">
+                <hardwareInterface>EffortJointInterface</hardwareInterface>
+                <mechanicalReduction>1</mechanicalReduction>
+            </actuator>
+            </transmission>
+        </xacro:macro>
+        <xacro:m_transmission index="1" joint_name="link1_bracket_1"/>
+        <xacro:m_transmission index="2" joint_name="link_2_bracket_2_1"/>
+        <xacro:m_transmission index="3" joint_name="bracket_2_2_link_3"/>
+        <xacro:m_transmission index="4" joint_name="bracket_3_2_link_4"/>
+        <xacro:m_transmission index="5" joint_name="link_5_link_6"/>
+        <xacro:m_transmission index="6" joint_name="link_6_left_gripper"/>
+        <xacro:m_transmission index="7" joint_name="link_6_right_gripper"/>
+        <gazebo>
+            <plugin name="gazebo_ros_control" filename="libgazebo_ros_control.so"/>
+        </gazebo>
 </robot>
